Commit message: add taco dataset

File: assets/rm65_leap_right/rm65_leap_left.urdf (robot description, URDF)
Before this commit: robot rm65_leap_right, 24 links, 23 joints
Links:
- added link index_tip_head
- added link middle_tip_head
- added link ring_tip_head
- added link thumb_tip_head
Joints:
- added joint index_tip: type floating, parent fingertip, child index_tip_head, origin xyz=0 -0.048 0.015 rpy=0 0 0
- added joint middle_tip: type floating, parent fingertip_2, child middle_tip_head, origin xyz=0 -0.048 0.015 rpy=0 0 0
- added joint ring_tip: type floating, parent fingertip_3, child ring_tip_head, origin xyz=0 -0.048 0.015 rpy=0 0 0
- added joint thumb_tip: type floating, parent thumb_fingertip, child thumb_tip_head, origin xyz=0 -0.06 -0.015 rpy=0 0 0

File: assets/rm65_leap_right/rm65_leap_right.urdf (robot description, URDF)
Before this commit: robot rm65_leap_right, 24 links, 23 joints
Links:
- added link index_tip_head
- added link middle_tip_head
- added link ring_tip_head
- added link thumb_tip_head
Joints:
- added joint index_tip: type floating, parent fingertip, child index_tip_head, origin xyz=0 -0.048 0.015 rpy=0 0 0
- added joint middle_tip: type floating, parent fingertip_2, child middle_tip_head, origin xyz=0 -0.048 0.015 rpy=0 0 0
- added joint ring_tip: type floating, parent fingertip_3, child ring_tip_head, origin xyz=0 -0.048 0.015 rpy=0 0 0
- added joint thumb_tip: type floating, parent thumb_fingertip, child thumb_tip_head, origin xyz=0 -0.06 -0.015 rpy=0 0 0
