Commit message: first bvdex codes

File: assets/rm65_leap_right/rm65_leap_left_m1.urdf (robot description, URDF)
Before this commit: robot rm65_leap_right, 29 links, 28 joints
Joints:
- joint arm_hand_joint: origin xyz=0 0 0.025 rpy=-1.5708 0 -1.5708 -> xyz=0 0 0.045 rpy=-1.5708 0 -1.5708
- joint palm_joint: origin xyz=0 0 0 rpy=-1.5708 0 0 -> xyz=0 0.02 0 rpy=-1.5708 0 0

File: assets/rm65_leap_right/rm65_leap_right_m1.urdf (robot description, URDF)
Before this commit: robot rm65_leap_right, 29 links, 28 joints
Joints:
- joint arm_hand_joint: origin xyz=0 0 0.025 rpy=1.5708 3.1415 0 -> xyz=0 0 0.045 rpy=1.5708 3.1415 0
- joint palm_joint: origin xyz=0 0 0 rpy=-1.5708 3.1415 0 -> xyz=0 0.02 0 rpy=-1.5708 3.1415 0

Commit message: huge modification

File: assets/rm65_leap_right/rm65_leap_left_m1.urdf (robot description, URDF)
Before this commit: robot rm65_leap_right, 29 links, 28 joints
Joints:
- joint palm_joint: origin xyz=0 0.02 0 rpy=-1.5708 0 0 -> xyz=0 0.02 0 rpy=-1.57079 0 0

File: rl_policy/taco_dataset/dex_retargeting/configs/teleop/leap_hand_left.urdf (robot description, URDF)
Before this commit: robot leap_left, 22 links, 21 joints
Links:
- removed link palm_lower_left
- removed link thumb_left_temp_base
- added link palm_lower, mass 0.237; collision mesh filename=meshes/palm_lower.stl scale=1 -1 1; visual mesh filename=meshes/palm_lower.stl scale=1 -1 1
- added link pip_4, mass 0.032; collision mesh filename=meshes/pip.stl scale=1 -1 1; visual mesh filename=meshes/pip.stl scale=1 -1 1
- link dip: geometry collision mesh filename=meshes/dip.stl; visual mesh filename=meshes/dip.stl
- link dip_2: geometry collision mesh filename=meshes/dip.stl; visual mesh filename=meshes/dip.stl
- link dip_3: geometry collision mesh filename=meshes/dip.stl; visual mesh filename=meshes/dip.stl
- link fingertip: geometry collision mesh filename=meshes/fingertip.stl; visual mesh filename=meshes/fingertip.stl
- link fingertip_2: geometry collision mesh filename=meshes/fingertip.stl; visual mesh filename=meshes/fingertip.stl
- link fingertip_3: geometry collision mesh filename=meshes/fingertip.stl; visual mesh filename=meshes/fingertip.stl
- link mcp_joint: geometry collision mesh filename=meshes/mcp_joint.stl; visual mesh filename=meshes/mcp_joint.stl
- link mcp_joint_2: geometry collision mesh filename=meshes/mcp_joint.stl; visual mesh filename=meshes/mcp_joint.stl
- link mcp_joint_3: geometry collision mesh filename=meshes/mcp_joint.stl; visual mesh filename=meshes/mcp_joint.stl
- link pip: geometry collision mesh filename=meshes/pip.stl; visual mesh filename=meshes/pip.stl
- link pip_2: geometry collision mesh filename=meshes/pip.stl; visual mesh filename=meshes/pip.stl
- link pip_3: geometry collision mesh filename=meshes/pip.stl; visual mesh filename=meshes/pip.stl
- link thumb_dip: geometry collision mesh filename=meshes/thumb_dip.stl; visual mesh filename=meshes/thumb_dip.stl
- link thumb_fingertip: geometry collision mesh filename=meshes/thumb_fingertip.stl; visual mesh filename=meshes/thumb_fingertip.stl
- link thumb_pip: geometry collision mesh filename=meshes/thumb_pip.stl; visual mesh filename=meshes/thumb_pip.stl
Joints:
- removed joint base_joint
- added joint palm_joint: type fixed, parent base, child palm_lower, origin xyz=0 0.02 0 rpy=-1.57079 0 0
- joint 0: origin xyz=-0.0122 0.03810 0.01450 rpy=-1.57079 0 1.57079 -> xyz=-0.012200000000000007713 0.038099999999999994982 0.01450000000000000073 rpy=-1.570796326794896558 -1.0065212660796336576e-15 1.5707963267948943376
- joint 1: origin xyz=-0.0825 -0.0857 0.0078 rpy=1.57079 1.57079 0 -> xyz=0.0530952496528625457958 0.058057756134899472233 -0.00472240357846021927 rpy=1.5707963267948950037 1.5707963267948945596 0; parent palm_lower_left -> palm_lower
- joint 10: origin xyz=0.015 0.0143 -0.013 rpy=1.57079 -1.57079 0 -> xyz=0.014999999999999971689 0.014299999999999951639 -0.012999999999999959505 rpy=1.5707963267948958919 -1.570796326794896336 0
- joint 11: origin xyz=0 -0.03609 0.0002 rpy=0 0 0 -> xyz=9.7144514654701197287e-17 -0.036099999999999868305 0.00020000000000007511769 rpy=4.5935029425113685044e-17 -2.8730071914463799514e-16 1.5565411607615035382e-32
- joint 12: child thumb_left_temp_base -> pip_4; origin xyz=-0.1448 -0.0900 0.0049 rpy=0 1.57079 0 -> xyz=-0.009395249652862533996 -0.0348422438651005258004 -0.017622403578460215601 rpy=3.14 -1.57 0; parent palm_lower_left -> palm_lower
- joint 13: origin xyz=0 -0.0143 -0.013 rpy=-1.57079 -1.57079 0 -> xyz=-2.7755575615628913511e-17 0.014300000000000005415 -0.013000000000000011546 rpy=1.5707963267948958919 -1.570796326794896336 0; parent thumb_left_temp_base -> pip_4
- joint 14: origin xyz=0 0.0145 -0.017 rpy=-1.57079 0 0 -> xyz=0 0.014499999999999966041 -0.017000000000000053263 rpy=-1.570796326794896558 1.6050198443300131245e-46 -1.9721522630516624601e-31
- joint 15: origin xyz=0 0.0466 0.0002 rpy=0 0 3.14159 -> xyz=-1.249000902703301108e-16 0.046599999999999863753 0.00019999999999997710581 rpy=1.5063958491491781023e-44 5.4234187233935260503e-31 3.141592653589793116
- joint 2: origin xyz=0.015 0.0143 -0.013 rpy=1.57079 -1.57079 0 -> xyz=0.01499999999999996822 0.014299999999999904801 -0.012999999999999824196 rpy=1.5707963267948958919 -1.570796326794896336 0
- joint 3: origin xyz=0 -0.0361 0.0002 rpy=0 0 0 -> xyz=-4.0880582495572692636e-09 -0.036100004210367367397 0.00020000000000007858714 rpy=4.5935029425113685044e-17 -2.8730071914463794583e-16 4.4395481053923607589e-32
- joint 4: origin xyz=-0.0122 0.0381 0.0145 rpy=-1.57079 0 1.57079 -> xyz=-0.012200000000000019856 0.038099999999999981104 0.01450000000000000594 rpy=-1.570796326794896558 -1.0065212760057939085e-15 1.5707963267948943376
- joint 5: origin xyz=-0.0825 -0.0403 0.0078 rpy=1.57079 1.57079 0 -> xyz=0.0530952496528625388569 0.013392243865100525113 -0.004722403578460229678 rpy=1.570796326794896558 1.570796326794896558 0; parent palm_lower_left -> palm_lower
- joint 6: origin xyz=0.015 0.0143 -0.013 rpy=1.57079 -1.57079 0 -> xyz=0.014999999999999975159 0.014300000000000000211 -0.013000000000000018485 rpy=1.5707963267948958919 -1.570796326794896336 0
- joint 7: origin xyz=0 -0.0361 0.0002 rpy=0 0 0 -> xyz=1.0061396160665481148e-16 -0.036099999999999854428 0.00020000000000007858714 rpy=4.5935029425113654229e-17 -2.8730071914463794583e-16 1.4408183216511868558e-31
- joint 8: origin xyz=-0.0122 0.0381 0.0145 rpy=-1.57079 0 1.57079 -> xyz=-0.012200000000000004244 0.038100000000000001921 0.014499999999999999001 rpy=-1.570796326794896558 -1.0065212660796360242e-15 1.5707963267948943376
- joint 9: origin xyz=-0.0825 0.0051 0.0078 rpy=1.57079 1.57079 0 -> xyz=0.0530952454426398371343 -0.032842243865100515521 -0.004722407666402932774 rpy=1.5707963267948950037 1.5707963267948945596 0; parent palm_lower_left -> palm_lower

File: rl_policy/taco_dataset/dex_retargeting/configs/teleop/leap_hand_right.urdf (robot description, URDF)
Before this commit: robot leap_right, 22 links, 21 joints
Links:
- removed link thumb_temp_base
- added link pip_4, mass 0.032; collision mesh filename=meshes/pip.stl; visual mesh filename=meshes/pip.stl
- link dip: geometry collision mesh filename=meshes/dip.stl; visual mesh filename=meshes/dip.stl
- link dip_2: geometry collision mesh filename=meshes/dip.stl; visual mesh filename=meshes/dip.stl
- link dip_3: geometry collision mesh filename=meshes/dip.stl; visual mesh filename=meshes/dip.stl
- link fingertip: geometry collision mesh filename=meshes/fingertip.stl; visual mesh filename=meshes/fingertip.stl
- link fingertip_2: geometry collision mesh filename=meshes/fingertip.stl; visual mesh filename=meshes/fingertip.stl
- link fingertip_3: geometry collision mesh filename=meshes/fingertip.stl; visual mesh filename=meshes/fingertip.stl
- link mcp_joint: geometry collision mesh filename=meshes/mcp_joint.stl; visual mesh filename=meshes/mcp_joint.stl
- link mcp_joint_2: geometry collision mesh filename=meshes/mcp_joint.stl; visual mesh filename=meshes/mcp_joint.stl
- link mcp_joint_3: geometry collision mesh filename=meshes/mcp_joint.stl; visual mesh filename=meshes/mcp_joint.stl
- link palm_lower: geometry collision mesh filename=meshes/palm_lower.stl; visual mesh filename=meshes/palm_lower.stl
- link pip: geometry collision mesh filename=meshes/pip.stl; visual mesh filename=meshes/pip.stl
- link pip_2: geometry collision mesh filename=meshes/pip.stl; visual mesh filename=meshes/pip.stl
- link pip_3: geometry collision mesh filename=meshes/pip.stl; visual mesh filename=meshes/pip.stl
- link thumb_dip: geometry collision mesh filename=meshes/thumb_dip.stl; visual mesh filename=meshes/thumb_dip.stl
- link thumb_fingertip: geometry collision mesh filename=meshes/thumb_fingertip.stl; visual mesh filename=meshes/thumb_fingertip.stl
- link thumb_pip: geometry collision mesh filename=meshes/thumb_pip.stl; visual mesh filename=meshes/thumb_pip.stl
Joints:
- removed joint base_joint
- added joint palm_joint: type fixed, parent base, child palm_lower, origin xyz=0 0.02 0 rpy=-1.5708 3.1415 0
- joint 0: origin xyz=-0.0122 0.03810 0.01450 rpy=-1.57079 0 1.57079 -> xyz=-0.012200000000000007713 0.038099999999999994982 0.01450000000000000073 rpy=-1.570796326794896558 -1.0065212660796336576e-15 1.5707963267948943376
- joint 1: origin xyz=-0.0070 0.0230 -0.0187 rpy=1.57079 1.57079 0 -> xyz=0.0530952496528625457958 0.058057756134899472233 -0.00472240357846021927 rpy=1.5707963267948950037 1.5707963267948945596 0
- joint 10: origin xyz=0.015 0.0143 -0.013 rpy=1.57079 -1.57079 0 -> xyz=0.014999999999999971689 0.014299999999999951639 -0.012999999999999959505 rpy=1.5707963267948958919 -1.570796326794896336 0
- joint 11: origin xyz=0 -0.03609 0.0002 rpy=0 0 0 -> xyz=9.7144514654701197287e-17 -0.036099999999999868305 0.00020000000000007511769 rpy=4.5935029425113685044e-17 -2.8730071914463799514e-16 1.5565411607615035382e-32
- joint 12: child thumb_temp_base -> pip_4; origin xyz=-0.0693 -0.0012 -0.0216 rpy=0 1.57079 0 -> xyz=-0.009395249652862533996 0.0342422438651005258004 -0.017622403578460215601 rpy=-8.2381766464939424156e-17 1.5707963267948956698 0
- joint 13: origin xyz=0 0.0143 -0.013 rpy=1.57079 -1.57079 0 -> xyz=-2.7755575615628913511e-17 0.014300000000000005415 -0.013000000000000011546 rpy=1.5707963267948958919 -1.570796326794896336 0; parent thumb_temp_base -> pip_4
- joint 14: origin xyz=0 0.0145 -0.017 rpy=-1.57079 0 0 -> xyz=0 0.014499999999999966041 -0.017000000000000053263 rpy=-1.570796326794896558 1.6050198443300131245e-46 -1.9721522630516624601e-31
- joint 15: origin xyz=0 0.0466 0.0002 rpy=0 0 3.14159 -> xyz=-1.249000902703301108e-16 0.046599999999999863753 0.00019999999999997710581 rpy=1.5063958491491781023e-44 5.4234187233935260503e-31 3.141592653589793116
- joint 2: origin xyz=0.015 0.0143 -0.013 rpy=1.57079 -1.57079 0 -> xyz=0.01499999999999996822 0.014299999999999904801 -0.012999999999999824196 rpy=1.5707963267948958919 -1.570796326794896336 0
- joint 3: origin xyz=0 -0.0361 0.0002 rpy=0 0 0 -> xyz=-4.0880582495572692636e-09 -0.036100004210367367397 0.00020000000000007858714 rpy=4.5935029425113685044e-17 -2.8730071914463794583e-16 4.4395481053923607589e-32
- joint 4: origin xyz=-0.0122 0.0381 0.0145 rpy=-1.57079 0 1.57079 -> xyz=-0.012200000000000019856 0.038099999999999981104 0.01450000000000000594 rpy=-1.570796326794896558 -1.0065212760057939085e-15 1.5707963267948943376
- joint 5: origin xyz=-0.0071 -0.0224 -0.0187 rpy=1.57079 1.57079 0 -> xyz=0.0530952496528625388569 0.013392243865100525113 -0.004722403578460229678 rpy=1.570796326794896558 1.570796326794896558 0
- joint 6: origin xyz=0.015 0.0143 -0.013 rpy=1.57079 -1.57079 0 -> xyz=0.014999999999999975159 0.014300000000000000211 -0.013000000000000018485 rpy=1.5707963267948958919 -1.570796326794896336 0
- joint 7: origin xyz=0 -0.0361 0.0002 rpy=0 0 0 -> xyz=1.0061396160665481148e-16 -0.036099999999999854428 0.00020000000000007858714 rpy=4.5935029425113654229e-17 -2.8730071914463794583e-16 1.4408183216511868558e-31
- joint 8: origin xyz=-0.0122 0.0381 0.0145 rpy=-1.57079 0 1.57079 -> xyz=-0.012200000000000004244 0.038100000000000001921 0.014499999999999999001 rpy=-1.570796326794896558 -1.0065212660796360242e-15 1.5707963267948943376
- joint 9: origin xyz=-0.00709 -0.0678 -0.0187 rpy=1.57079 1.57079 0 -> xyz=0.0530952454426398371343 -0.032842243865100515521 -0.004722407666402932774 rpy=1.5707963267948950037 1.5707963267948945596 0
